Commit message: add mobile robot design

File: urdf/manipulator.urdf (robot description, URDF)
Before this commit: robot manipulator, 8 links, 7 joints
Links:
- removed link gripper_rotor
- added link dummy_link
- added link front_left_shaft, mass 0.53535991363154; collision mesh filename=package://manipulator/meshes/front_left_shaft.STL; visual mesh filename=package://manipulator/meshes/front_left_shaft.STL
- added link front_left_wheel, mass 0.627305726641925; collision mesh filename=package://manipulator/meshes/front_left_wheel.STL; visual mesh filename=package://manipulator/meshes/front_left_wheel.STL
- added link front_right_shaft, mass 0.535359913631541; collision mesh filename=package://manipulator/meshes/front_right_shaft.STL; visual mesh filename=package://manipulator/meshes/front_right_shaft.STL
- added link front_right_wheel, mass 0.627305726641923; collision mesh filename=package://manipulator/meshes/front_right_wheel.STL; visual mesh filename=package://manipulator/meshes/front_right_wheel.STL
- added link gripper, mass 0.318053344407251; collision mesh filename=package://manipulator/meshes/gripper.STL; visual mesh filename=package://manipulator/meshes/gripper.STL
- added link manipulator_base, mass 0.343652649470195; collision mesh filename=package://manipulator/meshes/manipulator_base.STL; visual mesh filename=package://manipulator/meshes/manipulator_base.STL
- added link rear_left_wheel, mass 0.627305726641925; collision mesh filename=package://manipulator/meshes/rear_left_wheel.STL; visual mesh filename=package://manipulator/meshes/rear_left_wheel.STL
- added link rear_right_wheel, mass 0.627305726641921; collision mesh filename=package://manipulator/meshes/rear_right_wheel.STL; visual mesh filename=package://manipulator/meshes/rear_right_wheel.STL
- added link rear_shaft, mass 1.02790122650355; collision mesh filename=package://manipulator/meshes/rear_shaft.STL; visual mesh filename=package://manipulator/meshes/rear_shaft.STL
- link base_link: mass 0.343652649470198 -> 31.440945977861
- link gripper_left: mass 0.0811562982935575 -> 0.0811562982935577
- link gripper_right: mass 0.0811562982935573 -> 0.0811562982935572
- link link4: mass 1.48027818375282 -> 1.48027855179196
Joints:
- removed joint gripper_rotor_joint
- added joint dummy_joint: type fixed, parent dummy_link, child base_link, origin xyz=0 0 0 rpy=0 0 0, axis 0 0 0
- added joint front_left_shaft_joint: type continuous, parent base_link, child front_left_shaft, origin xyz=0.253321518968875 0.101599846414384 0.1016 rpy=0 0 1.5707963267949, axis 0 0 1
- added joint front_left_wheel_joint: type fixed, parent front_left_shaft, child front_left_wheel, origin xyz=0.1524 0 -3.76960577197494E-05 rpy=-1.5707963267949 0 -1.5707963267949, axis -1 0 0
- added joint front_right_shaft_joint: type continuous, parent base_link, child front_right_shaft, origin xyz=0.253321518968875 -0.101600153585616 0.1016 rpy=0 0 1.5707963267949, axis 0 0 1
- added joint front_right_wheel_joint: type fixed, parent front_right_shaft, child front_right_wheel, origin xyz=-0.1524 0 -3.76960577197494E-05 rpy=-1.5707963267949 0 -1.5707963267949, axis 0 1 0
- added joint gripper_joint: type continuous, parent link4, child gripper, origin xyz=0.248853265309693 0.00336707133293568 -0.0909728912537893 rpy=0 0.575281631239788 1.5707963267949, axis 0.0005742505150447 -0.999999765788382 0.000372370147822085
- added joint manipulator_base_joint: type fixed, parent base_link, child manipulator_base, origin xyz=0.354921518968873 -0.00035241085596216 0.2667 rpy=0 0 1.5707963267949, axis 0 0 0
- added joint rear_left_wheel_joint: type fixed, parent rear_shaft, child rear_left_wheel, origin xyz=0 0 0.508 rpy=0 0 0, axis 0 0 -1
- added joint rear_right_wheel_joint: type continuous, parent rear_shaft, child rear_right_wheel, origin xyz=0 0 0 rpy=0 0 0, axis 0 0 -1
- added joint rear_shaft_joint: type continuous, parent base_link, child rear_shaft, origin xyz=-0.254678481031125 -0.254000153585616 0.1016 rpy=-1.5707963267949 0 0, axis 0 0 -1
- joint gripper_left_joint: limit lower=0 upper=0 effort=0 velocity=0 -> lower=0.45 upper=-1.15 effort=10 velocity=1000; origin xyz=0.0018917 -0.02081 0.15152 rpy=-1.4737 -0.00030682 -1.5676 -> xyz=0.0127004769785455 -0.000826963988762031 -0.0208624359755367 rpy=-1.57079632680667 1.57042395663749 -1.57022207621871; parent gripper_rotor -> gripper
- joint gripper_right_joint: limit lower=0 upper=0 effort=0 velocity=0 -> lower=0.15 upper=-1.39 effort=10 velocity=1000; origin xyz=0.0017603 0.020915 0.15151 rpy=1.4737 0.00030682 1.5739 -> xyz=0.012700468056301 -0.00081142668143086 0.0208630053929066 rpy=1.57079632680667 -1.57042395663749 1.57137057737108; parent gripper_rotor -> gripper
- joint link1_joint: axis 0.015477 0 0.99988 -> -0.082237947023427 0 0.996612723212669; origin xyz=0 0 0.083058 rpy=0 -0.015478 -2.5461 -> xyz=0 0 0.083058 rpy=0 0.0823309272452037 1.4401673322326; parent base_link -> manipulator_base
- joint link2_joint: limit lower=0 upper=0 effort=0 velocity=0 -> lower=1.86 upper=-2.18 effort=10 velocity=1000; origin xyz=0.0015332 -0.0889 0.099048 rpy=1.5708 0 0 -> xyz=-0.0081465 -0.0889 0.098724 rpy=1.5708 0 0
- joint link3_joint: limit lower=0 upper=0 effort=0 velocity=0 -> lower=3.14 upper=-0.14 effort=10 velocity=1000
- joint link4_joint: limit lower=0 upper=0 effort=0 velocity=0 -> lower=2.35 upper=-1.77 effort=10 velocity=1000; origin xyz=0.30479 -0.0027849 0 rpy=0 0 0 -> xyz=0.29629 -0.071513 0 rpy=0 0 0
